Commit message: wip for gazebo

File: scout_description/urdf/mini.xacro (robot description, xacro)
@@ -174,4 +174,16 @@
         <child link="camera_link" />
     </joint>
+    <link name="inertial_link">
+        <inertial>
+            <mass value="132.3898489950015" />
+            <origin xyz=" 0 0 0" />
+            <inertia ixx="0.185196122711036" ixy="4.30144213829512E-08" ixz="5.81037523686401E-08" iyy="0.364893736238929" iyz="-0.000386720198091934" izz="0.223868521722778" />
+        </inertial>
+    </link>
+    <joint name="inertial_joint" type="fixed">
+        <origin xyz="0 0 0" rpy="0 0 0" />
+        <parent link="base_link" />
+        <child link="inertial_link" />
+    </joint>
 <!--
     <link name="inertial_link">

Commit message: wip for gazebo

File: scout_description/urdf/mini.xacro (robot description, xacro)
@@ -4,8 +4,4 @@
     <xacro:arg name="robot_namespace" default="/" />
     <xacro:arg name="urdf_extras" default="empty.urdf" />
-    <xacro:include filename="$(find scout_description)/urdf/scout_mini_wheel_1.xacro" />
-    <xacro:include filename="$(find scout_description)/urdf/scout_mini_wheel_2.xacro" />
-    <xacro:include filename="$(find scout_description)/urdf/scout_mini_wheel_3.xacro" />
-    <xacro:include filename="$(find scout_description)/urdf/scout_mini_wheel_4.xacro" />
     <!-- Variables -->
     <xacro:property name="M_PI" value="3.14159"/>
@@ -174,22 +170,9 @@
         <child link="camera_link" />
     </joint>
-    <link name="inertial_link">
+    <!-- <link name="inertial_link">
         <inertial>
             <mass value="132.3898489950015" />
             <origin xyz=" 0 0 0" />
             <inertia ixx="0.185196122711036" ixy="4.30144213829512E-08" ixz="5.81037523686401E-08" iyy="0.364893736238929" iyz="-0.000386720198091934" izz="0.223868521722778" />
-        </inertial>
-    </link>
-    <joint name="inertial_joint" type="fixed">
-        <origin xyz="0 0 0" rpy="0 0 0" />
-        <parent link="base_link" />
-        <child link="inertial_link" />
-    </joint>
-<!--
-    <link name="inertial_link">
-        <inertial>
-            <mass value="60" />
-            <origin xyz="0.0 0.0 0.0" />
-            <inertia ixx="2.288641" ixy="0" ixz="0" iyy="5.103976" iyz="0" izz="3.431465" />
         </inertial>
     </link>
@@ -206,31 +189,105 @@
         <child link="base_link"/>
     </joint> -->
-    <!-- Scout wheel macros -->
-    <!-- wheel labeled from 0 to 3, conter-clockwise, starting from front right wheel -->
-    <!-- motor 1 and 2 (left side) are mechanically installed in a reversed direction -->
-    <xacro:scout_mini_wheel_1 wheel_prefix="front_left" wheel_diameter="${wheel_diameter}" wheel_width="${wheel_width}">
-    <!--<origin
-            xyz="0 0 0"
-            rpy="0 0 0" />-->
-        <origin xyz="${wheelbase/2} ${track/2} ${wheel_vertical_offset}" rpy="-1.57 0 0" />
-    </xacro:scout_mini_wheel_1>
-    <xacro:scout_mini_wheel_2 wheel_prefix="rear_left" wheel_diameter="${wheel_diameter}" wheel_width="${wheel_width}">
-    <!--<origin
-            xyz="0 0 0"
-            rpy="0 0 0" />-->
-        <origin xyz="${-wheelbase/2} ${track/2} ${wheel_vertical_offset}" rpy="-1.57 0 0" />
-    </xacro:scout_mini_wheel_2>
-    <xacro:scout_mini_wheel_3 wheel_prefix="front_right" wheel_diameter="${wheel_diameter}" wheel_width="${wheel_width}">
-    <!--<origin
-            xyz="0 0 0"
-            rpy="0 0 0" />-->
-        <origin xyz="${wheelbase/2} ${-track/2} ${wheel_vertical_offset+0.001}" rpy="1.57 0 0" />
-    </xacro:scout_mini_wheel_3>
-    <xacro:scout_mini_wheel_4 wheel_prefix="rear_right" wheel_diameter="${wheel_diameter}" wheel_width="${wheel_width}">
-    <!--<origin
-           xyz="0 0 0"
-           rpy="0 0 0" />-->
-        <origin xyz="${-wheelbase/2} ${-track/2} ${wheel_vertical_offset+0.001}" rpy="1.57 0 0" />
-    </xacro:scout_mini_wheel_4>
+    <!-- Scout wheel -->
+    <link name="front_right_wheel_link">
+        <inertial>
+            <mass value="3" />
+            <origin xyz="0 0 0" />
+            <inertia ixx="0.7171" ixy="0" ixz="0" iyy="0.7171" iyz="0" izz="0.1361" />
+        </inertial>
+        <visual>
+            <origin xyz="0 0 0" rpy="0 0 0" />
+            <geometry>
+                <mesh filename="package://scout_description/meshes/wheel.dae" />
+            </geometry>
+        </visual>
+        <collision>
+            <origin xyz="0 0 0" rpy="0 0 0" />
+            <geometry>
+                <mesh filename="package://scout_description/meshes/wheel.dae" />
+            </geometry>
+        </collision>
+    </link>
+    <joint name="front_right_wheel" type="continuous">
+        <origin rpy="1.57 0 0" xyz="0.2319755 -0.2082515 -0.099998" />
+        <parent link="base_link" />
+        <child link="front_right_wheel_link" />
+        <axis xyz="0 0 -1" rpy="0 0 0" />
+    </joint>
+    <link name="front_left_wheel_link">
+        <inertial>
+            <mass value="3" />
+            <origin xyz="0 0 0" />
+            <inertia ixx="0.7171" ixy="0" ixz="0" iyy="0.7171" iyz="0" izz="0.1361" />
+        </inertial>
+        <visual>
+            <origin xyz="0 0 0" rpy="0 0 0" />
+            <geometry>
+                <mesh filename="package://scout_description/meshes/wheel.dae" />
+            </geometry>
+        </visual>
+        <collision>
+            <origin xyz="0 0 0" rpy="0 0 0" />
+            <geometry>
+                <mesh filename="package://scout_description/meshes/wheel.dae" />
+            </geometry>
+        </collision>
+    </link>
+    <joint name="front_left_wheel" type="continuous">
+        <origin rpy="-1.57 0 0" xyz="0.2319755 0.2082515 -0.100998" />
+        <parent link="base_link" />
+        <child link="front_left_wheel_link" />
+        <axis xyz="0 0 1" rpy="0 0 0" />
+    </joint>
+    <link name="rear_right_wheel_link">
+        <inertial>
+            <mass value="3" />
+            <origin xyz="0 0 0" />
+            <inertia ixx="0.7171" ixy="0" ixz="0" iyy="0.7171" iyz="0" izz="0.1361" />
+        </inertial>
+        <visual>
+            <origin xyz="0 0 0" rpy="0 0 0" />
+            <geometry>
+                <mesh filename="package://scout_description/meshes/wheel.dae" />
+            </geometry>
+        </visual>
+        <collision>
+            <origin xyz="0 0 0" rpy="0 0 0" />
+            <geometry>
+                <mesh filename="package://scout_description/meshes/wheel.dae" />
+            </geometry>
+        </collision>
+    </link>
+    <joint name="rear_right_wheel" type="continuous">
+        <origin rpy="1.57 0 0" xyz="-0.2319755 -0.2082515 -0.099998" />
+        <parent link="base_link" />
+        <child link="rear_right_wheel_link" />
+        <axis xyz="0 0 -1" rpy="0 0 0" />
+    </joint>
+    <link name="rear_left_wheel_link">
+        <inertial>
+            <mass value="3" />
+            <origin xyz="0 0 0" />
+            <inertia ixx="0.7171" ixy="0" ixz="0" iyy="0.7171" iyz="0" izz="0.1361" />
+        </inertial>
+        <visual>
+            <origin xyz="0 0 0" rpy="0 0 0" />
+            <geometry>
+                <mesh filename="package://scout_description/meshes/wheel.dae" />
+            </geometry>
+        </visual>
+        <collision>
+            <origin xyz="0 0 0" rpy="0 0 0" />
+            <geometry>
+                <mesh filename="package://scout_description/meshes/wheel.dae" />
+            </geometry>
+        </collision>
+    </link>
+    <joint name="rear_left_wheel" type="continuous">
+        <origin rpy="-1.57 0 0" xyz="-0.2319755 0.2082515 -0.100998" />
+        <parent link="base_link" />
+        <child link="rear_left_wheel_link" />
+        <axis xyz="0 0 1" rpy="0 0 0" />
+    </joint>
     <!-- Additional definitions -->
     <xacro:include filename="$(arg urdf_extras)" />

Commit message: Many changes to set up Gazebo sensors

File: scout_description/urdf/mini.xacro (robot description, xacro)
@@ -4,4 +4,8 @@
     <xacro:arg name="robot_namespace" default="/" />
     <xacro:arg name="urdf_extras" default="empty.urdf" />
+    <xacro:include filename="$(find scout_description)/urdf/scout_mini_wheel_1.xacro" />
+    <xacro:include filename="$(find scout_description)/urdf/scout_mini_wheel_2.xacro" />
+    <xacro:include filename="$(find scout_description)/urdf/scout_mini_wheel_3.xacro" />
+    <xacro:include filename="$(find scout_description)/urdf/scout_mini_wheel_4.xacro" />
     <!-- Variables -->
     <xacro:property name="M_PI" value="3.14159"/>
@@ -54,5 +58,5 @@
             <origin
                 xyz="0.0 0.0 0.0"
-                rpy="0 0 0" />
+                rpy="0 0 3.14159" />
             <mass
                 value="5" />
@@ -68,9 +72,9 @@
             <origin
                     xyz="0.0 0.0 0.0"
-                    rpy="0.0 0.0 3.14" />
-            <geometry>
-                <mesh filename="package://scout_description/meshes/box_link.STL" />
-            </geometry>
-            <material name = "red">
+                    rpy="0.0 0.0 0.0" />
+            <geometry>
+                <mesh filename="package://scout_description/meshes/box-parts/box.stl" />
+            </geometry>
+            <material name = "white">
             <color rgba="1 1 1 1" />
             </material>
@@ -86,9 +90,35 @@
     </link>
     <joint name="box_joint" type="fixed">
-        <origin xyz="0 0 0.055" rpy="0 0 3.14" />
+        <origin xyz="0 0 0.055" rpy="0 0 0" />
         <parent link="base_link" />
         <child link="box_link" />
     </joint>
  <link name="laser_link">
+        <visual>
+            <origin
+                    xyz="0.0 0.0 0.0"
+                    rpy="0.0 0.0 0.0" />
+            <geometry>
+                <mesh filename="package://scout_description/meshes/box-parts/lidar.stl" />
+            </geometry>
+            <material name = "cyan">
+            <color rgba="0 0.5 1 1" />
+            </material>
+        </visual>
+        <collision>
+            <origin
+                    xyz="0 0 0.31"
+                    rpy="0 0 0" />
+          <geometry>
+                    <cylinder radius="0.06" length="0.1"/>
+          </geometry>
+        </collision>
+    </link>
+    <joint name="laser_joint" type="fixed">
+        <origin xyz="0.015732 -0.001804 0.200816" rpy="0 0 0" />
+        <parent link="box_link" />
+        <child link="laser_link" />
+    </joint>
+ <link name="camera_link">
         <inertial>
             <origin
@@ -110,8 +140,8 @@
                     rpy="0.0 0.0 0.0" />
             <geometry>
-                    <cylinder radius="0.01" length="0.01"/>
+                <mesh filename="package://scout_description/meshes/box-parts/camera.stl" />
             </geometry>
             <material name = "red">
-            <color rgba="1 1 1 1" />
+            <color rgba="1 0 0 1" />
             </material>
         </visual>
@@ -121,14 +151,21 @@
                     rpy="0 0 0" />
           <geometry>
-                    <cylinder radius="0.06" length="0.1"/>
-          </geometry>
-        </collision>
-    </link>
-    <joint name="laser_joint" type="fixed">
-        <origin xyz="0 0 0.23" rpy="0 0 0" />
-        <parent link="base_link" />
-        <child link="laser_link" />
-    </joint>
- <link name="camera_link">
+                    <box size="0.01 0.01 0.01"/>
+          </geometry>
+        </collision>
+    </link>
+    <joint name="camera_joint" type="fixed">
+        <origin xyz="0.192646 -0.001255 0.096" rpy="0 0 0" />
+        <parent link="box_link" />
+        <child link="camera_link" />
+    </joint>
+    <link name="camera_optical_link">
+    </link>
+    <joint name="camera_optical_joint" type="fixed">
+        <origin xyz="0.01495 0 0.0125" rpy="0 0 0" />
+        <parent link="camera_link" />
+        <child link="camera_optical_link" />
+    </joint>
+ <link name="monitor_link">
         <inertial>
             <origin
@@ -150,36 +187,24 @@
                     rpy="0.0 0.0 0.0" />
             <geometry>
+                <mesh filename="package://scout_description/meshes/box-parts/monitor.stl" />
+            </geometry>
+            <material name = "purple">
+            <color rgba="1 0 1 1" />
+            </material>
+        </visual>
+        <collision>
+            <origin
+                    xyz="0 0 0.31"
+                    rpy="0 0 0" />
+          <geometry>
                     <box size="0.01 0.01 0.01"/>
-            </geometry>
-            <material name = "red">
-            <color rgba="1 1 1 1" />
-            </material>
-        </visual>
-        <collision>
-            <origin
-                    xyz="0 0 0.31"
-                    rpy="0 0 0" />
-          <geometry>
-                    <box size="0.01 0.01 0.01"/>
-          </geometry>
-        </collision>
-    </link>
-    <joint name="camera_joint" type="fixed">
-        <origin xyz="0.2 0 0.16" rpy="0 0 0" />
-        <parent link="base_link" />
-        <child link="camera_link" />
-    </joint>
-    <!-- <link name="inertial_link">
-        <inertial>
-            <mass value="132.3898489950015" />
-            <origin xyz=" 0 0 0" />
-            <inertia ixx="0.185196122711036" ixy="4.30144213829512E-08" ixz="5.81037523686401E-08" iyy="0.364893736238929" iyz="-0.000386720198091934" izz="0.223868521722778" />
-        </inertial>
-    </link>
-    <joint name="inertial_joint" type="fixed">
-        <origin xyz="0 0 0" rpy="0 0 0" />
-        <parent link="base_link" />
-        <child link="inertial_link" />
-    </joint> -->
+          </geometry>
+        </collision>
+    </link>
+    <joint name="monitor_joint" type="fixed">
+        <origin xyz="-0.088892 -0.001255 0.101303" rpy="0 0 0" />
+        <parent link="box_link" />
+        <child link="monitor_link" />
+    </joint>
     <!-- For testing, hang the robot up in the air -->
     <!-- <link name="world" />
@@ -189,105 +214,31 @@
         <child link="base_link"/>
     </joint> -->
-    <!-- Scout wheel -->
-    <link name="front_right_wheel_link">
-        <inertial>
-            <mass value="3" />
-            <origin xyz="0 0 0" />
-            <inertia ixx="0.7171" ixy="0" ixz="0" iyy="0.7171" iyz="0" izz="0.1361" />
-        </inertial>
-        <visual>
-            <origin xyz="0 0 0" rpy="0 0 0" />
-            <geometry>
-                <mesh filename="package://scout_description/meshes/wheel.dae" />
-            </geometry>
-        </visual>
-        <collision>
-            <origin xyz="0 0 0" rpy="0 0 0" />
-            <geometry>
-                <mesh filename="package://scout_description/meshes/wheel.dae" />
-            </geometry>
-        </collision>
-    </link>
-    <joint name="front_right_wheel" type="continuous">
-        <origin rpy="1.57 0 0" xyz="0.2319755 -0.2082515 -0.099998" />
-        <parent link="base_link" />
-        <child link="front_right_wheel_link" />
-        <axis xyz="0 0 -1" rpy="0 0 0" />
-    </joint>
-    <link name="front_left_wheel_link">
-        <inertial>
-            <mass value="3" />
-            <origin xyz="0 0 0" />
-            <inertia ixx="0.7171" ixy="0" ixz="0" iyy="0.7171" iyz="0" izz="0.1361" />
-        </inertial>
-        <visual>
-            <origin xyz="0 0 0" rpy="0 0 0" />
-            <geometry>
-                <mesh filename="package://scout_description/meshes/wheel.dae" />
-            </geometry>
-        </visual>
-        <collision>
-            <origin xyz="0 0 0" rpy="0 0 0" />
-            <geometry>
-                <mesh filename="package://scout_description/meshes/wheel.dae" />
-            </geometry>
-        </collision>
-    </link>
-    <joint name="front_left_wheel" type="continuous">
-        <origin rpy="-1.57 0 0" xyz="0.2319755 0.2082515 -0.100998" />
-        <parent link="base_link" />
-        <child link="front_left_wheel_link" />
-        <axis xyz="0 0 1" rpy="0 0 0" />
-    </joint>
-    <link name="rear_right_wheel_link">
-        <inertial>
-            <mass value="3" />
-            <origin xyz="0 0 0" />
-            <inertia ixx="0.7171" ixy="0" ixz="0" iyy="0.7171" iyz="0" izz="0.1361" />
-        </inertial>
-        <visual>
-            <origin xyz="0 0 0" rpy="0 0 0" />
-            <geometry>
-                <mesh filename="package://scout_description/meshes/wheel.dae" />
-            </geometry>
-        </visual>
-        <collision>
-            <origin xyz="0 0 0" rpy="0 0 0" />
-            <geometry>
-                <mesh filename="package://scout_description/meshes/wheel.dae" />
-            </geometry>
-        </collision>
-    </link>
-    <joint name="rear_right_wheel" type="continuous">
-        <origin rpy="1.57 0 0" xyz="-0.2319755 -0.2082515 -0.099998" />
-        <parent link="base_link" />
-        <child link="rear_right_wheel_link" />
-        <axis xyz="0 0 -1" rpy="0 0 0" />
-    </joint>
-    <link name="rear_left_wheel_link">
-        <inertial>
-            <mass value="3" />
-            <origin xyz="0 0 0" />
-            <inertia ixx="0.7171" ixy="0" ixz="0" iyy="0.7171" iyz="0" izz="0.1361" />
-        </inertial>
-        <visual>
-            <origin xyz="0 0 0" rpy="0 0 0" />
-            <geometry>
-                <mesh filename="package://scout_description/meshes/wheel.dae" />
-            </geometry>
-        </visual>
-        <collision>
-            <origin xyz="0 0 0" rpy="0 0 0" />
-            <geometry>
-                <mesh filename="package://scout_description/meshes/wheel.dae" />
-            </geometry>
-        </collision>
-    </link>
-    <joint name="rear_left_wheel" type="continuous">
-        <origin rpy="-1.57 0 0" xyz="-0.2319755 0.2082515 -0.100998" />
-        <parent link="base_link" />
-        <child link="rear_left_wheel_link" />
-        <axis xyz="0 0 1" rpy="0 0 0" />
-    </joint>
+    <!-- Scout wheel macros -->
+    <!-- wheel labeled from 0 to 3, conter-clockwise, starting from front right wheel -->
+    <!-- motor 1 and 2 (left side) are mechanically installed in a reversed direction -->
+    <xacro:scout_mini_wheel_1 wheel_prefix="front_left" wheel_diameter="${wheel_diameter}" wheel_width="${wheel_width}">
+    <!--<origin
+            xyz="0 0 0"
+            rpy="0 0 0" />-->
+        <origin xyz="${wheelbase/2} ${track/2} ${wheel_vertical_offset}" rpy="-1.57 0 0" />
+    </xacro:scout_mini_wheel_1>
+    <xacro:scout_mini_wheel_2 wheel_prefix="rear_left" wheel_diameter="${wheel_diameter}" wheel_width="${wheel_width}">
+    <!--<origin
+            xyz="0 0 0"
+            rpy="0 0 0" />-->
+        <origin xyz="${-wheelbase/2} ${track/2} ${wheel_vertical_offset}" rpy="-1.57 0 0" />
+    </xacro:scout_mini_wheel_2>
+    <xacro:scout_mini_wheel_3 wheel_prefix="front_right" wheel_diameter="${wheel_diameter}" wheel_width="${wheel_width}">
+    <!--<origin
+            xyz="0 0 0"
+            rpy="0 0 0" />-->
+        <origin xyz="${wheelbase/2} ${-track/2} ${wheel_vertical_offset+0.001}" rpy="1.57 0 0" />
+    </xacro:scout_mini_wheel_3>
+    <xacro:scout_mini_wheel_4 wheel_prefix="rear_right" wheel_diameter="${wheel_diameter}" wheel_width="${wheel_width}">
+    <!--<origin
+           xyz="0 0 0"
+           rpy="0 0 0" />-->
+        <origin xyz="${-wheelbase/2} ${-track/2} ${wheel_vertical_offset+0.001}" rpy="1.57 0 0" />
+    </xacro:scout_mini_wheel_4>
     <!-- Additional definitions -->
     <xacro:include filename="$(arg urdf_extras)" />
