Commit message: Add diff drive controller (only drives, does not diff)

File: scout_description/urdf/mini.xacro (robot description, xacro)
@@ -4,8 +4,5 @@
     <xacro:arg name="robot_namespace" default="/" />
     <xacro:arg name="urdf_extras" default="empty.urdf" />
-    <xacro:include filename="$(find scout_description)/urdf/scout_mini_wheel_1.xacro" />
-    <xacro:include filename="$(find scout_description)/urdf/scout_mini_wheel_2.xacro" />
-    <xacro:include filename="$(find scout_description)/urdf/scout_mini_wheel_3.xacro" />
-    <xacro:include filename="$(find scout_description)/urdf/scout_mini_wheel_4.xacro" />
+    <xacro:include filename="$(find scout_description)/urdf/scout_mini_wheel.xacro" />
     <!-- Variables -->
     <xacro:property name="M_PI" value="3.14159"/>
@@ -217,28 +214,16 @@
     <!-- wheel labeled from 0 to 3, conter-clockwise, starting from front right wheel -->
     <!-- motor 1 and 2 (left side) are mechanically installed in a reversed direction -->
-    <xacro:scout_mini_wheel_1 wheel_prefix="front_left" wheel_diameter="${wheel_diameter}" wheel_width="${wheel_width}">
-    <!--<origin
-            xyz="0 0 0"
-            rpy="0 0 0" />-->
+    <xacro:scout_mini_wheel wheel_prefix="front_left" wheel_diameter="${wheel_diameter}" wheel_width="${wheel_width}" axis="1">
         <origin xyz="${wheelbase/2} ${track/2} ${wheel_vertical_offset}" rpy="-1.57 0 0" />
-    </xacro:scout_mini_wheel_1>
-    <xacro:scout_mini_wheel_2 wheel_prefix="rear_left" wheel_diameter="${wheel_diameter}" wheel_width="${wheel_width}">
-    <!--<origin
-            xyz="0 0 0"
-            rpy="0 0 0" />-->
+    </xacro:scout_mini_wheel>
+    <xacro:scout_mini_wheel wheel_prefix="rear_left" wheel_diameter="${wheel_diameter}" wheel_width="${wheel_width}" axis="1">
         <origin xyz="${-wheelbase/2} ${track/2} ${wheel_vertical_offset}" rpy="-1.57 0 0" />
-    </xacro:scout_mini_wheel_2>
-    <xacro:scout_mini_wheel_3 wheel_prefix="front_right" wheel_diameter="${wheel_diameter}" wheel_width="${wheel_width}">
-    <!--<origin
-            xyz="0 0 0"
-            rpy="0 0 0" />-->
+    </xacro:scout_mini_wheel>
+    <xacro:scout_mini_wheel wheel_prefix="front_right" wheel_diameter="${wheel_diameter}" wheel_width="${wheel_width}" axis="-1">
         <origin xyz="${wheelbase/2} ${-track/2} ${wheel_vertical_offset+0.001}" rpy="1.57 0 0" />
-    </xacro:scout_mini_wheel_3>
-    <xacro:scout_mini_wheel_4 wheel_prefix="rear_right" wheel_diameter="${wheel_diameter}" wheel_width="${wheel_width}">
-    <!--<origin
-           xyz="0 0 0"
-           rpy="0 0 0" />-->
+    </xacro:scout_mini_wheel>
+    <xacro:scout_mini_wheel wheel_prefix="rear_right" wheel_diameter="${wheel_diameter}" wheel_width="${wheel_width}" axis="-1">
         <origin xyz="${-wheelbase/2} ${-track/2} ${wheel_vertical_offset+0.001}" rpy="1.57 0 0" />
-    </xacro:scout_mini_wheel_4>
+    </xacro:scout_mini_wheel>
     <!-- Additional definitions -->
     <xacro:include filename="$(arg urdf_extras)" />

File: scout_description/urdf/scout_mini_wheel.xacro (robot description, xacro)
@@ -24,30 +24,54 @@
 -->
 <robot xmlns:xacro="http://ros.org/wiki/xacro" name="scout_wheel">
-    <xacro:macro name="scout_wheel_type2" params="wheel_prefix *joint_pose">
-        <link name="${wheel_prefix}_wheel_link">
+  <xacro:macro name="scout_mini_wheel" params="wheel_prefix wheel_diameter wheel_width axis *joint_pose">
+    <xacro:property name="wheel_radius" value="${wheel_diameter / 2}" />
+            <link name="${wheel_prefix}_wheel_link">
             <inertial>
                 <mass value="3" />
                 <origin xyz="0 0 0" />
-                <inertia ixx="0.7171" ixy="0" ixz="0" iyy="0.1361" iyz="0" izz="0.7171" />
-            </inertial>
+                <inertia
+                    ixx="0.006564" ixy="0" ixz="0"
+                    iyy="0.006564" iyz="0"
+                    izz="0.0096"/>
+              </inertial>
             <visual>
                 <origin xyz="0 0 0" rpy="0 0 0" />
                 <geometry>
-                    <mesh filename="package://scout_description/meshes/wheel_type1.dae" />
+                    <mesh filename="package://scout_description/meshes/wheel.dae" />
                 </geometry>
             </visual>
             <collision>
-                <origin xyz="0 0 0" rpy="${M_PI/2} 0 0" />
-                <geometry>
-                    <cylinder length="${wheel_length}" radius="${wheel_radius}" />
-                </geometry>
+              <origin
+                xyz="0 0 0.03"
+                rpy="0 0 0" />
+              <geometry>
+                <!-- <mesh
+                  filename="package://scout_description/meshes/wheel.dae" /> -->
+                  <cylinder radius="0.08" length="0.084"/>
+              </geometry>
             </collision>
         </link>
         <joint name="${wheel_prefix}_wheel" type="continuous">
+            <!--<origin
+                  xyz="0.14547 0.20835 -0.07424"
+                  rpy="0 1.57 0" />-->
             <parent link="base_link"/>
             <child link="${wheel_prefix}_wheel_link"/>
             <xacro:insert_block name="joint_pose"/>
-            <axis xyz="0 -1 0" rpy="0 0 0" />
+            <axis xyz="0 0 ${axis}" rpy="0 0 0" />
+            <dynamics damping="0.0" friction="0.0"/>
+            <limit effort="1000" velocity="20"/>  <!-- High limits for fast turns -->
         </joint>
+<gazebo reference="rear_left_wheel">
+  <mu1>200.0</mu1>  <!-- High for no longitudinal slip (propulsion) -->
+  <mu2>200.0</mu2>  <!-- High for lateral grip during turns (prevents sliding) -->
+  <slip1>0.01</slip1>  <!-- Small torsional slip for realism/stability -->
+  <slip2>0.01</slip2>  <!-- Lateral slip; tune higher (0.1) if turns feel too sticky -->
+  <kp>1e7</kp>      <!-- Stiffness: prevents sinking -->
+  <kd>10.0</kd>     <!-- Damping: reduces bounce; increased from 1.0 -->
+  <fdir1>1 0 0</fdir1>
+  <minDepth>0.005</minDepth>  <!-- Deeper contacts for better force transmission -->
+  <maxContacts>10</maxContacts>
+</gazebo>
     </xacro:macro>
 </robot>

Commit message: switch to diff_drive_controller

File: scout_description/urdf/mini.xacro (robot description, xacro)
@@ -3,5 +3,4 @@
     xmlns:xacro="http://ros.org/wiki/xacro">
     <xacro:arg name="robot_namespace" default="/" />
-    <xacro:arg name="urdf_extras" default="empty.urdf" />
     <xacro:include filename="$(find scout_description)/urdf/scout_mini_wheel.xacro" />
     <!-- Variables -->
@@ -91,5 +90,5 @@
         <child link="box_link" />
     </joint>
- <link name="laser_link">
+    <link name="laser_link">
         <visual>
             <origin
@@ -117,5 +116,5 @@
         <child link="laser_link" />
     </joint>
- <link name="camera_link">
+    <link name="camera_link">
         <inertial>
             <origin
@@ -164,5 +163,5 @@
         <child link="camera_optical_link" />
     </joint>
- <link name="monitor_link">
+    <link name="monitor_link">
         <inertial>
             <origin
@@ -204,11 +203,4 @@
         <child link="monitor_link" />
     </joint>
-    <!-- For testing, hang the robot up in the air -->
-    <!-- <link name="world" />
-    <joint name="world_to_base_link=" type="fixed">
-        <origin xyz="0 0 0.5" rpy="0 0 0" />
-        <parent link="world"/>
-        <child link="base_link"/>
-    </joint> -->
     <!-- Scout wheel macros -->
     <!-- wheel labeled from 0 to 3, conter-clockwise, starting from front right wheel -->
@@ -226,6 +218,41 @@
         <origin xyz="${-wheelbase/2} ${-track/2} ${wheel_vertical_offset+0.001}" rpy="1.57 0 0" />
     </xacro:scout_mini_wheel>
-    <!-- Additional definitions -->
-    <xacro:include filename="$(arg urdf_extras)" />
+    <ros2_control name="GazeboSimSystem" type="system">
+        <hardware>
+            <plugin>gz_ros2_control/GazeboSimSystem</plugin>
+        </hardware>
+        <joint name="front_left_wheel">
+	    <command_interface name="velocity">
+                <param name="min">-10.0</param>
+                <param name="max">10.0</param>
+            </command_interface>
+            <state_interface name="position"/>
+            <state_interface name="velocity"/>
+        </joint>
+        <joint name="rear_left_wheel">
+	    <command_interface name="velocity">
+                <param name="min">-10.0</param>
+                <param name="max">10.0</param>
+            </command_interface>
+            <state_interface name="position"/>
+            <state_interface name="velocity"/>
+        </joint>
+        <joint name="front_right_wheel">
+	    <command_interface name="velocity">
+                <param name="min">-10.0</param>
+                <param name="max">10.0</param>
+            </command_interface>
+            <state_interface name="position"/>
+            <state_interface name="velocity"/>
+        </joint>
+        <joint name="rear_right_wheel">
+	    <command_interface name="velocity">
+                <param name="min">-10.0</param>
+                <param name="max">10.0</param>
+            </command_interface>
+            <state_interface name="position"/>
+            <state_interface name="velocity"/>
+        </joint>
+    </ros2_control>
     <!-- Gazebo definitions  -->
     <xacro:include filename="$(find scout_description)/urdf/scout_mini.gazebo" />

File: scout_description/urdf/scout_mini_wheel.xacro (robot description, xacro)
@@ -63,15 +63,15 @@
             <limit effort="1000" velocity="20"/>  <!-- High limits for fast turns -->
         </joint>
-<gazebo reference="${wheel_prefix}_wheel_link">
-  <mu1>200.0</mu1>  <!-- High for no longitudinal slip (propulsion) -->
-  <mu2>0.75</mu2>  <!-- High for lateral grip during turns (prevents sliding) -->
-  <slip1>0.01</slip1>  <!-- Small torsional slip for realism/stability -->
-  <slip2>0.01</slip2>  <!-- Lateral slip; tune higher (0.1) if turns feel too sticky -->
-  <kp>1e7</kp>      <!-- Stiffness: prevents sinking -->
-  <kd>10.0</kd>     <!-- Damping: reduces bounce; increased from 1.0 -->
-  <fdir1>1 0 0</fdir1>
-  <minDepth>0.005</minDepth>  <!-- Deeper contacts for better force transmission -->
-  <maxContacts>10</maxContacts>
-</gazebo>
-    </xacro:macro>
+    <gazebo reference="${wheel_prefix}_wheel_link">
+      <mu1>200.0</mu1>  <!-- High for no longitudinal slip (propulsion) -->
+      <mu2>0.75</mu2>  <!-- High for lateral grip during turns (prevents sliding) -->
+      <slip1>0.01</slip1>  <!-- Small torsional slip for realism/stability -->
+      <slip2>0.01</slip2>  <!-- Lateral slip; tune higher (0.1) if turns feel too sticky -->
+      <kp>1e7</kp>      <!-- Stiffness: prevents sinking -->
+      <kd>10.0</kd>     <!-- Damping: reduces bounce; increased from 1.0 -->
+      <fdir1>1 0 0</fdir1>
+      <minDepth>0.005</minDepth>  <!-- Deeper contacts for better force transmission -->
+      <maxContacts>10</maxContacts>
+    </gazebo>
+  </xacro:macro>
 </robot>
