Commit message: move all gazebo related things into sim.gazebo

File: scout_description/urdf/scout_mini.xacro (robot description, xacro)
@@ -159,30 +159,5 @@
     <origin xyz="${-wheelbase/2} ${-track/2} ${wheel_vertical_offset}" rpy="${M_PI/2} 0 0"/>
   </xacro:wheel>
-  <ros2_control name="GazeboSimSystem" type="system">
-    <hardware>
-      <plugin>gz_ros2_control/GazeboSimSystem</plugin>
-    </hardware>
-    <joint name="front_left_wheel">
-      <command_interface name="velocity"/>
-      <state_interface name="position"/>
-      <state_interface name="velocity"/>
-    </joint>
-    <joint name="rear_left_wheel">
-      <command_interface name="velocity"/>
-      <state_interface name="position"/>
-      <state_interface name="velocity"/>
-    </joint>
-    <joint name="front_right_wheel">
-      <command_interface name="velocity"/>
-      <state_interface name="position"/>
-      <state_interface name="velocity"/>
-    </joint>
-    <joint name="rear_right_wheel">
-      <command_interface name="velocity"/>
-      <state_interface name="position"/>
-      <state_interface name="velocity"/>
-    </joint>
-  </ros2_control>
-  <!-- Gazebo definitions  -->
-  <xacro:include filename="$(find scout_description)/urdf/sensors.gazebo"/>
+  <!-- Gazebo sim definitions  -->
+  <xacro:include filename="$(find scout_description)/urdf/sim.gazebo"/>
 </robot>
